File: PCB/laya's macropad.kicad_sch (KiCad schematic)
At the start: 10 parts, among them J1 OLED_128x64, U2 MCU_Seeed_XIAO_RP2040

Commit message: oled changed
Parts:
- removed J1: OLED_128x64, ScottoKeebs_Components:OLED_128x64, symbol symbs:OLED_128x64
- added J1: OLED_128x32, ScottoKeebs_Components:OLED_128x32, symbol ScottoKeebs:OLED_128x32
Connections:
- net GND: now also J1.1 (GND)
- net at U2.12 (3V3): now also J1.2 (VCC)
- net at U2.5 (PA8_A4_D4_SDA): now also J1.4 (SDA)
- net at U2.6 (PA9_A5_D5_SCL): now also J1.3 (SCL)
Changed lines of the file:
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@@
 	(wire
 		(pts
-			(xy 156.21 71.12) (xy 156.21 72.39)
+			(xy 152.4 69.85) (xy 152.4 72.39)
 		)
 		(stroke
@@
 	(wire
 		(pts
-			(xy 156.21 72.39) (xy 158.75 72.39)
+			(xy 152.4 72.39) (xy 158.75 72.39)
 		)
 		(stroke
@@
 	(symbol
 		(lib_id "power:PWR_FLAG")
-		(at 156.21 71.12 0)
+		(at 152.4 69.85 0)
 		(unit 1)
 		(exclude_from_sim no)
@@
 		(fields_autoplaced yes)
 		(property "Reference" "#FLG01"
-			(at 156.21 69.215 0)
+			(at 152.4 67.945 0)
 			(effects
 				(font
@@
 		)
 		(property "Value" "PWR_FLAG"
-			(at 156.21 66.04 0)
+			(at 152.4 64.77 0)
 			(effects
 				(font
@@
 		)
 		(property "Footprint" ""
-			(at 156.21 71.12 0)
+			(at 152.4 69.85 0)
 			(effects
 				(font
@@
 		)
 		(property "Datasheet" "~"
-			(at 156.21 71.12 0)
+			(at 152.4 69.85 0)
 			(effects
 				(font
@@
 		)
 		(property "Description" "Special symbol for telling ERC where power comes from"
-			(at 156.21 71.12 0)
+			(at 152.4 69.85 0)
 			(effects
 				(font
@@
 	)
 	(symbol
-		(lib_id "symbs:OLED_128x64")
-		(at 166.37 46.99 180)
+		(lib_id "ScottoKeebs:OLED_128x32")
+		(at 166.37 46.99 90)
 		(unit 1)
 		(exclude_from_sim no)
@@
 		(fields_autoplaced yes)
 		(property "Reference" "J1"
-			(at 177.8 40.6399 0)
+			(at 172.72 38.0999 90)
 			(effects
 				(font
@@
 			)
 		)
-		(property "Value" "OLED_128x64"
-			(at 177.8 43.1799 0)
+		(property "Value" "OLED_128x32"
+			(at 172.72 40.6399 90)
 			(effects
 				(font
@@
 			)
 		)
-		(property "Footprint" "ScottoKeebs_Components:OLED_128x64"
-			(at 166.37 33.02 0)
+		(property "Footprint" "ScottoKeebs_Components:OLED_128x32"
+			(at 157.48 46.99 0)
 			(effects
 				(font
@@
 		)
 		(property "Datasheet" ""
-			(at 165.1 46.99 90)
+			(at 165.1 46.99 0)
 			(effects
 				(font
@@
 			)
 		)
+		(pin "4"
+		)
+		(pin "3"
+		)
 		(pin "2"
 		)
-		(pin "3"
-		)
 		(pin "1"
 		)
-		(pin "4"
-		)
 		(instances
